File: design_files/ASD2421.sch (EAGLE design)
At the start: 11 parts, among them J2 DF12-32-DS

Commit message: Update Rev and Format
Parts:
- removed U$3: AS-ITM-00133, tinycircuits:AS-ITM-00133
- removed U$4: AS-ITM-00134, tinycircuits:AS-ITM-00134
- removed U$5, U$6, U$7, U$8: AS-ITM-00135, tinycircuits:AS-ITM-00135
- added D2: ACSA02-41SURKWA-F01, tinycircuits:AS-ITM-00133
- added R1: 10.0K, tinycircuits:AS-ITM-00032
- added R2, R3, R4, R5: 330, tinycircuits:AS-ITM-00135
- added U1: SX1506, tinycircuits:AS-ITM-00134
- D1: value AS-ITM-00133 -> ACSA02-41SURKWA-F01; PARTNO (none) -> AS-ITM-00133
- renumbered U$2 to D1
Connections:
- new net RST: R1.1, U1.NRESET
- net AD4/SDA: now also U1.SDA; no longer U$4.SDA
- net AD5/SCL: now also U1.SCL; no longer U$4.SCL
- net GND: now also U1.GND, U1.GND2, U1.GND3, U1.GND4, U1.GNDPAD; no longer U$4.GND, U$4.GND2, U$4.GND3, U$4.GND4, U$4.GNDPAD
- net GPIO0: now also R5.6; no longer U$6.6
- net GPIO1: now also R5.8; no longer U$6.8
- net GPIO10: now also D2.C, R4.2; no longer U$3.C, U$5.2
- net GPIO11: now also D2.D, R4.4; no longer U$3.D, U$5.4
- net GPIO12: now also D2.E, R4.6; no longer U$3.E, U$5.6
- net GPIO13: now also D2.F, R4.8; no longer U$3.F, U$5.8
- net GPIO14: now also D2.G, R5.2; no longer U$3.G, U$6.2
- net GPIO15: now also D2.DP, R5.4; no longer U$3.DP, U$6.4
- net GPIO2: now also R3.7; no longer U$8.7
- net GPIO3: now also R3.5; no longer U$8.5
- net GPIO4: now also R3.3; no longer U$8.3
- net GPIO5: now also R3.1; no longer U$8.1
- net GPIO6: now also R2.7; no longer U$7.7
- net GPIO7: now also R2.5; no longer U$7.5
- net GPIO8: now also D2.A, R2.3; no longer U$3.A, U$7.3
- net GPIO9: now also D2.B, R2.1; no longer U$3.B, U$7.1
- net N$1: now also R2.2, U1.IO9; no longer U$4.IO9, U$7.2
- net N$10: now also R3.8, U1.IO2; no longer U$4.IO2, U$8.8
- net N$19: now also R4.1, U1.IO10; no longer U$4.IO10, U$5.1
- net N$2: now also R2.4, U1.IO8; no longer U$4.IO8, U$7.4
- net N$20: now also R4.3, U1.IO11; no longer U$4.IO11, U$5.3
- net N$21: now also R4.5, U1.IO12; no longer U$4.IO12, U$5.5
- net N$22: now also R4.7, U1.IO13; no longer U$4.IO13, U$5.7
- net N$23: now also R5.1, U1.IO14; no longer U$4.IO14, U$6.1
- net N$24: now also R5.3, U1.IO15; no longer U$4.IO15, U$6.3
- net N$25: now also R5.5, U1.IO0; no longer U$4.IO0, U$6.5
- net N$26: now also R5.7, U1.IO1; no longer U$4.IO1, U$6.7
- net N$3: now also R2.6, U1.IO7; no longer U$4.IO7, U$7.6
- net N$4: now also R2.8, U1.IO6; no longer U$4.IO6, U$7.8
- net N$6: now also R3.2, U1.IO5; no longer U$4.IO5, U$8.2
- net N$7: now also R3.4, U1.IO4; no longer U$4.IO4, U$8.4
- net N$9: now also R3.6, U1.IO3; no longer U$4.IO3, U$8.6
- net VCC: now also D2.VCC, D2.VCC1, R1.2, U1.VCC1, U1.VCC2, U1.VDDM; no longer U$3.VCC, U$3.VCC1, U$4.NINT, U$4.NRESET, U$4.VCC1, U$4.VCC2, U$4.VDDM
Other:
- note added: "2"
- note added: "7 Segment Displays"
- note added: "Hand Populated: -"
- note added: "Hand Soldered: -"
- note added: "Non Populated: -"
- note added: "Notes: -"
- note added: "SX1506 IO Expander"
- note added: "Variant: Standard"
- note removed: "1"
- moved on the sheet: C1, C2, C3
